Commit message: got urdf to spawn

File: install/six_dof_arm/share/six_dof_arm/urdf/six_dof_arm.urdf (robot description, URDF)
Before this commit: robot Assem1, 7 links, 6 joints
Links:
- removed link base_link
- removed link link_4_1
- removed link link_4_2
- added link link_5, mass 0.19053; collision mesh filename=package://six_dof_arm/meshes/link_5.STL; visual mesh filename=package://six_dof_arm/meshes/link_5.STL
- added link link_6, mass 0.11653; collision mesh filename=package://six_dof_arm/meshes/link_6.STL; visual mesh filename=package://six_dof_arm/meshes/link_6.STL
- added link link_7, mass 0.11653; collision mesh filename=package://six_dof_arm/meshes/link_7.STL; visual mesh filename=package://six_dof_arm/meshes/link_7.STL
- added link stand, mass 17.147; collision mesh filename=package://six_dof_arm/meshes/base_link.STL; visual mesh filename=package://six_dof_arm/meshes/base_link.STL
- link link_1: mass 2.3084 -> 3.0905; geometry collision mesh filename=package://six_dof_arm/meshes/link_1.STL; visual mesh filename=package://six_dof_arm/meshes/link_1.STL
- link link_2: mass 0.91528 -> 5.5867; geometry collision mesh filename=package://six_dof_arm/meshes/link_2.STL; visual mesh filename=package://six_dof_arm/meshes/link_2.STL
- link link_3: mass 1.9287 -> 2.8262; geometry collision mesh filename=package://six_dof_arm/meshes/link_3.STL; visual mesh filename=package://six_dof_arm/meshes/link_3.STL
- link link_4: mass 0.39086 -> 1.8097; geometry collision mesh filename=package://six_dof_arm/meshes/link_4.STL; visual mesh filename=package://six_dof_arm/meshes/link_4.STL
Joints:
- removed joint joint_0
- removed joint joint_4_1
- removed joint joint_4_2
- added joint joint_4: type revolute, parent link_3, child link_4, origin xyz=-0.35 0 0 rpy=0 0 1.5708, axis 0 0 1, limit lower=0 upper=3.142 effort=200 velocity=3
- added joint joint_5: type revolute, parent link_4, child link_5, origin xyz=-0.188 0 0 rpy=0 0 0, axis 1 0 0, limit lower=0 upper=3.142 effort=200 velocity=3
- added joint joint_6: type prismatic, parent link_5, child link_6, origin xyz=0.54 -0.4 0 rpy=0 0 0, axis 0 0 -1, limit lower=0 upper=0.03 effort=100 velocity=3
- added joint joint_7: type prismatic, parent link_5, child link_7, origin xyz=0.54 0.4 0 rpy=3.1416 0 0, axis 0 0 1, limit lower=-0.03 upper=0 effort=100 velocity=3
- joint joint_1: child link_2 -> link_1; limit lower=-3.14159 upper=3.14159 effort=1 velocity=1 -> lower=0 upper=3.142 effort=300 velocity=3; origin xyz=-0.15 0.16 -0.01 rpy=-1.5249 0.0328 -2.1913 -> xyz=0 0 0.2 rpy=1.5708 0 1.5708; parent link_1 -> stand
- joint joint_2: child link_3 -> link_2; limit lower=-3.14159 upper=3.14159 effort=1 velocity=1 -> lower=-1.57 upper=1.57 effort=200 velocity=3; origin xyz=-0.35014 0.001494 0.00019501 rpy=1.5708 -0.94986 3.1416 -> xyz=0 0.205 0 rpy=0 0 0; parent link_2 -> link_1
- joint joint_3: axis 1 0 0 -> 0 0 1; child link_4 -> link_3; limit lower=-3.14159 upper=3.14159 effort=1 velocity=1 -> lower=0 upper=3.142 effort=200 velocity=3; origin xyz=0.35909 0.043643 0.0018034 rpy=0.25066 1.5295 1.5708 -> xyz=0 0.4 0 rpy=0 0 0; parent link_3 -> link_2

File: src/six_dof_arm/urdf/six_dof_arm.urdf (robot description, URDF)
Before this commit: robot robot_arm_urdf, 8 links, 7 joints
Links:
- removed link base_link
- added link stand, mass 17.147; collision mesh filename=package://six_dof_arm/meshes/base_link.STL; visual mesh filename=package://six_dof_arm/meshes/base_link.STL
- link link_1: geometry collision mesh filename=package://six_dof_arm/meshes/link_1.STL; visual mesh filename=package://six_dof_arm/meshes/link_1.STL
- link link_2: geometry collision mesh filename=package://six_dof_arm/meshes/link_2.STL; visual mesh filename=package://six_dof_arm/meshes/link_2.STL
- link link_3: geometry collision mesh filename=package://six_dof_arm/meshes/link_3.STL; visual mesh filename=package://six_dof_arm/meshes/link_3.STL
- link link_4: geometry collision mesh filename=package://six_dof_arm/meshes/link_4.STL; visual mesh filename=package://six_dof_arm/meshes/link_4.STL
- link link_5: geometry collision mesh filename=package://six_dof_arm/meshes/link_5.STL; visual mesh filename=package://six_dof_arm/meshes/link_5.STL
- link link_6: geometry collision mesh filename=package://six_dof_arm/meshes/link_6.STL; visual mesh filename=package://six_dof_arm/meshes/link_6.STL
- link link_7: geometry collision mesh filename=package://six_dof_arm/meshes/link_7.STL; visual mesh filename=package://six_dof_arm/meshes/link_7.STL
Joints:
- joint joint_1: parent base_link -> stand
- joint joint_4: limit lower=0 upper=-3.142 effort=200 velocity=3 -> lower=0 upper=3.142 effort=200 velocity=3

Commit message: added non working files

File: install/six_dof_arm/share/six_dof_arm/urdf/six_dof_arm.urdf (robot description, URDF)
Before this commit: robot six_dof_arm, 8 links, 7 joints
Links:
- removed link stand
- added link base_link, mass 17.147; collision mesh filename=package://six_dof_arm/meshes/base_link.STL; visual mesh filename=package://six_dof_arm/meshes/base_link.STL
Joints:
- joint joint_1: parent stand -> base_link
- joint joint_3: limit lower=0 upper=3.142 effort=200 velocity=3 -> lower=-1.5 upper=1.5 effort=200 velocity=3
- joint joint_4: limit lower=0 upper=3.142 effort=200 velocity=3 -> lower=-3.142 upper=0 effort=200 velocity=3
