Commit message: finished manipulation

File: install/my_cubes_pkg/share/my_cubes_pkg/models/urdf/blue_cube.urdf (robot description, URDF)
Before this commit: robot blue_cube, 1 links, 0 joints
Links:
- link base_link: geometry collision box size=0.05 0.05 0.05; visual box size=0.05 0.05 0.05

File: install/my_cubes_pkg/share/my_cubes_pkg/models/urdf/green_cube.urdf (robot description, URDF)
Before this commit: robot green_cube, 1 links, 0 joints
Links:
- link base_link: geometry collision box size=0.05 0.05 0.05; visual box size=0.05 0.05 0.05

File: install/my_cubes_pkg/share/my_cubes_pkg/models/urdf/red_cube.urdf (robot description, URDF)
Before this commit: robot red_cube, 1 links, 0 joints
Links:
- link base_link: geometry collision box size=0.05 0.05 0.05; visual box size=0.05 0.05 0.05

File: install/my_robot_pkg/share/my_robot_pkg/description/xacro/panda_ros2control.xacro (robot description, xacro)
@@ -152,49 +152,53 @@
     <gazebo reference="panda_link0">
       <selfCollide>false</selfCollide>
-      <material>Gazebo/Orange</material>
+      <material>Gazebo/White</material>
     </gazebo>
     <gazebo reference="panda_link1">
       <selfCollide>false</selfCollide>
-      <material>Gazebo/Orange</material>
+      <material>Gazebo/White</material>
     </gazebo>
     <gazebo reference="panda_link2">
       <selfCollide>false</selfCollide>
-      <material>Gazebo/Orange</material>
+      <material>Gazebo/White</material>
     </gazebo>
     <gazebo reference="panda_link3">
       <selfCollide>false</selfCollide>
-      <material>Gazebo/Orange</material>
+      <material>Gazebo/White</material>
     </gazebo>
     <gazebo reference="panda_link4">
       <selfCollide>false</selfCollide>
-      <material>Gazebo/Orange</material>
+      <material>Gazebo/White</material>
     </gazebo>
     <gazebo reference="panda_link5">
       <selfCollide>false</selfCollide>
-      <material>Gazebo/Orange</material>
+      <material>Gazebo/White</material>
     </gazebo>
     <gazebo reference="panda_link6">
       <selfCollide>false</selfCollide>
-      <material>Gazebo/Orange</material>
+      <material>Gazebo/White</material>
     </gazebo>
     <gazebo reference="panda_link7">
       <selfCollide>false</selfCollide>
-      <material>Gazebo/Orange</material>
+      <material>Gazebo/White</material>
     </gazebo>
     <gazebo reference="panda_link8">
       <selfCollide>false</selfCollide>
-      <material>Gazebo/Orange</material>
+      <material>Gazebo/White</material>
     </gazebo>
     <gazebo reference="panda_hand">
       <selfCollide>false</selfCollide>
-      <material>Gazebo/Orange</material>
+      <material>Gazebo/White</material>
     </gazebo>
     <gazebo reference="panda_leftfinger">
       <selfCollide>false</selfCollide>
-      <material>Gazebo/Orange</material>
+      <material>Gazebo/White</material>
+      <mu1>3.0</mu1> <!-- Coefficient of friction -->
+      <mu2>3.0</mu2>
     </gazebo>
     <gazebo reference="panda_rightfinger">
       <selfCollide>false</selfCollide>
-      <material>Gazebo/Orange</material>
+      <material>Gazebo/White</material>
+      <mu1>3.0</mu1> <!-- Coefficient of friction -->
+      <mu2>3.0</mu2>
     </gazebo>
     <gazebo reference="end_effector_frame_fixed_joint">
